File: PowerShield.kicad_pcb (KiCad board)
At the start: 2 copper layers, 50 x 50 mm, 24 parts, among them J1 XT60PW-M

Commit message: V2
Parts:
- moved C1 3.92 mm to (6.43, 0.00), turned to 0 degrees
- moved C3 3.49 mm to (16.9, -3.50), turned to 0 degrees
Routing:
- net VCC: track 3494.6 -> 3492.0 mm
Other:
- board text added: "BOOT"
- board text added: "Phoque Power Shield North"
- board text added: "RESET"
- board text added: "To flash: hold boot and press reset Mount using brass standoffs PCB resistor not for prolonged brakes"
- board text added: "XT60"
